File: series-prop/receiver-v0.1.0/receiver-v0.1.0.kicad_pcb (KiCad board)
At the start: 2 copper layers, 47 x 84.9 mm, 67 parts, among them IC1 LM66200DRLR, J1 Conn_01x17, J10 Conn_01x03_Pin, J11 Conn_01x04_Pin, J13 USB_C_Receptacle_USB2.0_16P, J2 Conn_01x04_Pin, J4 Conn_01x17, J5 Conn_01x01_Pin, J6 Screw_Terminal_01x02, J7 Screw_Terminal_01x03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

Commit message: added remote design files
Parts:
- added D2: SMF5V0A, Diode_SMD:D_SMF, F.Cu at (132.3, 65.5)
- added U8: TPD4EUSB30, Package_SON:USON-10_2.5x1.0mm_P0.5mm, F.Cu at (130.9, 68.4)
Routing:
- net Net-(J13-CC2): track 4.97 -> 15.4 mm, vias 0 -> 2
- net /USB_P: track 40.8 -> 48.8 mm, vias 1 -> 2
- net VBUS: track 29.6 -> 36.8 mm
- net /USB_N: track 45.4 -> 52.3 mm, vias 1 -> 2
- net GND: track 39.5 -> 44.7 mm
- net Net-(J13-CC1): track 5.29 -> 9.28 mm
Other:
- board text added: "ESD"
- board text added: "TVS"
- board text added: "Warning: GPIO 14 is level-shifted to 5V at the terminal block Warning: Use internal pullup resistor for the CONFIG button connected to GPIO3 and the ENTER button connected to GPIO15"
- board text removed: "Warning: GPIO 14 is level-shifted to 5V at the terminal block Warning: Use internal pullup resistor for the ENTER button connected to GPIO3 and GPIO15"
