File: series-prop/remote-v0.1.0/remote-v0.1.0.kicad_pcb (KiCad board)
At the start: 2 copper layers, 47 x 84.9 mm, 67 parts, among them IC1 LM66200DRLR, J1 Conn_01x17, J10 Conn_01x03_Pin, J11 Conn_01x04_Pin, J13 USB_C_Receptacle_USB2.0_16P, J2 Conn_01x04_Pin, J4 Conn_01x17, J5 Conn_01x01_Pin, J6 Screw_Terminal_01x02, J7 Screw_Terminal_01x03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

Commit message: added remote design files
Parts:
- removed C18, C26: 10u, Capacitor_SMD:C_1206_3216Metric
- removed C19: 100n, Capacitor_SMD:C_0603_1608Metric
- removed C20, C22: 22u, Capacitor_SMD:C_0805_2012Metric
- removed L2: 4.7u, Inductor_SMD:L_Sunlord_SWPA4030S
- removed R21: 10k, Resistor_SMD:R_0603_1608Metric
- removed U6: 74AHCT1G125, Package_TO_SOT_SMD:SOT-23-5
- removed U7: 3544-2, PicoLume:3544-2
- added C4: 10u, Capacitor_SMD:C_0603_1608Metric, F.Cu at (114.2, 80.2)
- added C5: 22u, Capacitor_SMD:C_0805_2012Metric, F.Cu at (122.0, 89.0)
- added D2: SMF5V0A, Diode_SMD:D_SMF, F.Cu at (130.3, 73.9)
- added D3: LED, LED_SMD:LED_0603_1608Metric, F.Cu at (117.9, 86.0)
- added D4: LED, LED_SMD:LED_0603_1608Metric, F.Cu at (114.9, 76.7)
- added J12: Screw_Terminal_01x02, TerminalBlock:TerminalBlock_bornier-2_P5.08mm, F.Cu at (142.5, 93.8)
- added J14: Conn_01x15, Connector_PinHeader_2.54mm:PinHeader_1x15_P2.54mm_Vertical, F.Cu at (144.8, 103.5)
- added J3: Conn_01x02_Pin, Connector_JST:JST_PH_S2B-PH-K_1x02_P2.00mm_Horizontal, F.Cu at (135.3, 69.5)
- added R12: 10k, Resistor_SMD:R_0603_1608Metric, F.Cu at (116.5, 76.7)
- added R13: 10k, Resistor_SMD:R_0603_1608Metric, F.Cu at (116.3, 85.9)
- added R14: 10k, Resistor_SMD:R_0603_1608Metric, F.Cu at (119.5, 80.8)
- added R17: 5k, Resistor_SMD:R_0603_1608Metric, F.Cu at (120.9, 76.7)
- IC1: value LM66200DRLR -> BQ25185DLHR; footprint PicoLume:LM66200DRLR -> PicoLume:SON40P220X200X80-11N
- J1: value Conn_01x17 -> Conn_01x02_Pin; footprint Connector_PinHeader_2.54mm:PinHeader_1x17_P2.54mm_Vertical -> Connector_PinHeader_2.54mm:PinHeader_1x02_P2.54mm_Vertical
- J7: value Screw_Terminal_01x03 -> Screw_Terminal_01x02; footprint TerminalBlock:TerminalBlock_bornier-3_P5.08mm -> TerminalBlock:TerminalBlock_bornier-2_P5.08mm
- R15: value 330R -> 1k
- U5: value AP63205WU -> TPD4EUSB30; footprint Package_TO_SOT_SMD:TSOT-23-6 -> Package_SON:USON-10_2.5x1.0mm_P0.5mm
- moved R15 36.9 mm to (119.3, 76.7)
- moved J1 25.0 mm to (136.6, 74.6)
- moved F2 11.3 mm to (136.5, 81.3), turned to -90 degrees
- moved U5 10.6 mm to (125.5, 74.2), turned to 0 degrees
- moved C1 8.05 mm to (122.0, 91.0), turned to 0 degrees
- moved G*** 7.18 mm to (123.5, 80.5)
- moved IC1 5.23 mm to (116.3, 81.0), turned to 90 degrees
- moved G*** 3.54 mm to (129.4, 82.5)
- moved R11 1.95 mm to (127.8, 73.1), turned to 90 degrees
Connections:
- F2 pad 1: Net-(U5-EN) -> Net-(J1-Pin_2)
- IC1 pad 1: GND -> VSYS
- IC1 pad 2: +5V -> VBAT
- IC1 pad 3: VIN -> Net-(IC1-STAT2)
- IC1 pad 6: +5V_BUCK -> Net-(IC1-TS/MR)
- IC1 pad 7: +5V -> Net-(IC1-ILIM/VSET)
- IC1 pad 8: Net-(IC1-ST) -> Net-(IC1-ISET)
- J1 pad 1: +5V -> Net-(J1-Pin_1)
- J1 pad 2: /GPIO29_ADC3 -> Net-(J1-Pin_2)
- J6 pad 1: VBAT -> Net-(J1-Pin_1)
- J6 pad 2: GND -> Net-(J1-Pin_2)
- J7 pad 2: FUSED -> /GPIO3
- R15 pad 1: /GPIO14 -> GND
- R15 pad 2: Net-(R15-Pad2) -> Net-(IC1-ISET)
- U1 pad 1: +5V -> VSYS
- U1 pad 3: +5V -> VSYS
- U5 pad 1: +5V_BUCK -> /USB_P
- U5 pad 2: Net-(U5-EN) -> /USB_N
- U5 pad 3: Net-(U5-EN) -> GND
- U5 pad 4: GND -> Net-(J13-CC1)
- U5 pad 5: Net-(U5-SW) -> Net-(J13-CC2)
- U5 pad 6: Net-(U5-BST) -> unconnected-(U5-NC-Pad6)
Routing:
- net /GPIO3: track 61.2 -> 138.1 mm
- net +5V: track 45.3 -> 0.00 mm, vias 2 -> 0
- net VSYS: track 0.00 -> 29.1 mm, vias 0 -> 2
- net /GPIO15: track 57.2 -> 84.6 mm
- net Net-(R15-Pad2): track 25.5 -> 0.00 mm, vias 2 -> 0
- net +5V_BUCK: track 21.6 -> 0.00 mm, vias 2 -> 0
- net /GPIO29_ADC3: track 14.3 -> 0.00 mm
- net FUSED: track 13.4 -> 0.00 mm
- net Net-(J1-Pin_1): track 0.00 -> 12.2 mm
- net Net-(U5-EN): track 11.7 -> 0.00 mm, vias 2 -> 0
- net Net-(U5-SW): track 9.59 -> 0.00 mm
- net Net-(J1-Pin_2): track 0.00 -> 9.02 mm
- net VIN: track 19.8 -> 12.2 mm
- net Net-(J13-CC2): track 4.97 -> 11.8 mm, vias 0 -> 2
- net VBUS: track 29.6 -> 35.7 mm
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Other:
- board text added: "+"
- board text added: "-"
- board text added: "5k"
- board text added: "BAT+"
- board text added: "BATTERY JUMPER"
- board text added: "CHG"
- board text added: "ESD"
- board text added: "F2"
- board text added: "Fault"
- board text added: "PicoLume Remote picolume.com v0.1.0"
- board text added: "PicoLume Remote v0.1.0"
- board text added: "TVS"
- board text added: "VBAT"
- board text added: "Warning: Use internal pullup resistor for the CONFIG button connected to GPIO3 and the ENTER button connected to GPIO15"
- board text removed: "29"
- board text removed: "330"
- board text removed: "4.7uH"
- board text removed: "5V"
- board text removed: "6V-30V"
- board text removed: "GPIO14"
- board text removed: "LM"
- board text removed: "POS"
- board text removed: "POS 6V-30V"
- board text removed: "POS FUSED"
- board text removed: "PicoLume Receiver picolume.com v0.1.0"
- board text removed: "PicoLume Reciever v0.1.0"
- board text removed: "Warning: GPIO 14 is level-shifted to 5V at the terminal block Warning: Use internal pullup resistor for the ENTER button connected to GPIO3 and GPIO15"
